File: projeto-pcb/pcb-atividade/pcb-atividade.kicad_pcb (KiCad board)
At the start: 2 copper layers, 7 parts, among them J1 Conn_01x02_Socket, J3 Conn_01x04_Pin, Q1 BC414, U1 Pico

Commit message: feat: altering the circuit
Parts:
- removed J3: Conn_01x04_Pin, Connector_PinHeader_1.27mm:PinHeader_1x04_P1.27mm_Vertical
- added J2: Conn_01x02_Socket, Connector_PinHeader_1.27mm:PinHeader_1x02_P1.27mm_Vertical, F.Cu at (146.5, 90.2)
Connections:
- Q1 pad 1: Net-(J3-Pin_2) -> Net-(J2-Pin_2)
- Q1 pad 2: Net-(J3-Pin_2) -> Net-(Q1-B)
- R2 pad 2: Net-(J3-Pin_2) -> Net-(Q1-B)
Routing:
- net VCC: track 79.1 -> 16.0 mm
- net Net-(J3-Pin_2): track 21.8 -> 0.00 mm
- net Net-(J2-Pin_2): track 0.00 -> 13.8 mm
- net Net-(Q1-B): track 0.00 -> 8.27 mm
- net VCC_Led: track 29.3 -> 29.9 mm
